File: StepUp_module_12to450V.kicad_sch (KiCad schematic)
At the start: 0 parts

Commit message: DBG18
Other:
- note added: "Randomsone"
- note removed: "Randoms"
Changed lines of the file:
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@@
 		)
 	)
-	(text "Randoms"
+	(text "Randomsone"
 		(exclude_from_sim no)
 		(at 135.89 27.94 0)

Commit message: Preping release 1.0.0
Other:
- note removed: "Randomsone"
Changed lines of the file:
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@@
-		)
-	)
-	(text "Randomsone"
-		(exclude_from_sim no)
-		(at 135.89 27.94 0)
-		(effects
-			(font
-				(size 5.08 5.08)
-			)
 		)
 	)

Commit message: Solving rev hist
Other:
- note added: "."
Changed lines of the file:
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@@
+		)
+	)
+	(text "."
+		(exclude_from_sim no)
+		(at 381 304.8 0)
+		(effects
+			(font
+				(size 1.27 1.27)
+			)
 		)
 	)

Commit message: Solving rev hist again
Other:
- note added: ".."
- note removed: "."
Changed lines of the file:
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@@
 		)
 	)
-	(text "."
+	(text ".."
 		(exclude_from_sim no)
 		(at 381 304.8 0)

Commit message: Rev hist update
Other:
- note added: "..."
- note removed: ".."
Changed lines of the file:
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@@
 		)
 	)
-	(text ".."
+	(text "..."
 		(exclude_from_sim no)
 		(at 381 304.8 0)

Commit message: General notes added
Other:
- note added: "NOTE STYLING CONVENTION"
- note removed: "..."
- note removed: "CHECKED - DRC completed, schematic and layout ready for review."
- note removed: "Comment"
- note removed: "DESIGN CONSIDERATIONS"
- note removed: "DRAFT - Early concept stage, schematic drafted."
- note removed: "NOTES"
- note removed: "Not fitted components are marked as"
- note removed: "PRELIMINARY - Minor schematic changes are expected, ready for layout planning."
- note removed: "RELEASED - Design ready for manufacturing."

Commit message: Ready to release
Other:
- note added: "Status: ${VARIANT}"
- note removed: "${SHEET_NAME_10}"
- note removed: "${SHEET_NAME_5}"
- note removed: "${SHEET_NAME_6}"
- note removed: "${SHEET_NAME_7}"
- note removed: "${SHEET_NAME_8}"
- note removed: "${SHEET_NAME_9}"
- note removed: "10"
- note removed: "5"
- note removed: "6"
- note removed: "7"
- note removed: "8"
- note removed: "9"
- note removed: "Variant: ${VARIANT}"
Changed lines of the file:
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@@
 		(comment 9 "NA")
 	)
-	(text "Variant: ${VARIANT}"
+	(text "Status: ${VARIANT}"
 		(exclude_from_sim no)
 		(at 25.4 58.42 0)
@@
 		)
 	)
-	(text "${SHEET_NAME_5}"
-		(exclude_from_sim no)
-		(at 45.72 114.3 0)
-		(effects
-			(font
-				(face "Times New Roman")
-				(size 4 4)
-				(color 0 0 0 1)
-			)
-			(justify left bottom)
-			(href "#7")
-		)
-	)
-	(text "7"
-		(exclude_from_sim no)
-		(at 35.56 129.54 0)
-		(effects
-			(font
-				(face "Times New Roman")
-				(size 4 4)
-				(color 0 0 0 1)
-			)
-			(justify right bottom)
-			(href "#7")
-		)
-	)
-	(text "${SHEET_NAME_8}"
-		(exclude_from_sim no)
-		(at 45.72 137.16 0)
-		(effects
-			(font
-				(face "Times New Roman")
-				(size 4 4)
-				(color 0 0 0 1)
-			)
-			(justify left bottom)
-			(href "#8")
-		)
-	)
-	(text "10"
-		(exclude_from_sim no)
-		(at 35.56 152.4 0)
-		(effects
-			(font
-				(face "Times New Roman")
-				(size 4 4)
-				(color 0 0 0 1)
-			)
-			(justify right bottom)
-			(href "#10")
-		)
-	)
 	(text "${SHEET_NAME_2}"
 		(exclude_from_sim no)
@@
 			(justify right bottom)
 			(href "#1")
-		)
-	)
-	(text "${SHEET_NAME_6}"
-		(exclude_from_sim no)
-		(at 45.72 121.92 0)
-		(effects
-			(font
-				(face "Times New Roman")
-				(size 4 4)
-				(color 0 0 0 1)
-			)
-			(justify left bottom)
-			(href "#6")
 		)
 	)
@@
 		)
 	)
-	(text "${SHEET_NAME_7}"
-		(exclude_from_sim no)
-		(at 45.72 129.54 0)
-		(effects
-			(font
-				(face "Times New Roman")
-				(size 4 4)
-				(color 0 0 0 1)
-			)
-			(justify left bottom)
-			(href "#7")
-		)
-	)
-	(text "5"
-		(exclude_from_sim no)
-		(at 35.56 114.3 0)
-		(effects
-			(font
-				(face "Times New Roman")
-				(size 4 4)
-				(color 0 0 0 1)
-			)
-			(justify right bottom)
-			(href "#5")
-		)
-	)
 	(text "${BOARD_NAME}"
 		(exclude_from_sim no)
@@
 			(justify left bottom)
 			(href "#1")
-		)
-	)
-	(text "${SHEET_NAME_9}"
-		(exclude_from_sim no)
-		(at 45.72 144.78 0)
-		(effects
-			(font
-				(face "Times New Roman")
-				(size 4 4)
-				(color 0 0 0 1)
-			)
-			(justify left bottom)
-			(href "#9")
-		)
-	)
-	(text "8"
-		(exclude_from_sim no)
-		(at 35.56 137.16 0)
-		(effects
-			(font
-				(face "Times New Roman")
-				(size 4 4)
-				(color 0 0 0 1)
-			)
-			(justify right bottom)
-			(href "#8")
 		)
 	)
@@
 		)
 	)
-	(text "${SHEET_NAME_10}"
-		(exclude_from_sim no)
-		(at 45.72 152.4 0)
-		(effects
-			(font
-				(face "Times New Roman")
-				(size 4 4)
-				(color 0 0 0 1)
-			)
-			(justify left bottom)
-			(href "#10")
-		)
-	)
 	(text "Index"
 		(exclude_from_sim no)
@@
 		)
 	)
-	(text "6"
-		(exclude_from_sim no)
-		(at 35.56 121.92 0)
-		(effects
-			(font
-				(face "Times New Roman")
-				(size 4 4)
-				(color 0 0 0 1)
-			)
-			(justify right bottom)
-			(href "#6")
-		)
-	)
 	(text "${SHEET_NAME_4}"
 		(exclude_from_sim no)
@@
 		)
 	)
-	(text "9"
-		(exclude_from_sim no)
-		(at 35.56 144.78 0)
-		(effects
-			(font
-				(face "Times New Roman")
-				(size 4 4)
-				(color 0 0 0 1)
-			)
-			(justify right bottom)
-			(href "#9")
-		)
-	)
