File: Revision History.kicad_sch (KiCad schematic)
At the start: 0 parts

Commit message: testing lib issue
Changed lines of the file:
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@@
 		(rev "${REVISION}")
 		(company "${COMPANY}")
+		(comment 1 "\"Comment 1\"")
+		(comment 2 "\"Comment 2\"")
+		(comment 3 "\"Comment 3\"")
+		(comment 4 "\"Comment 4\"")
+		(comment 5 "\"Comment 5\"")
+		(comment 6 "\"Comment 6\"")
+		(comment 7 "\"Comment 7\"")
+		(comment 8 "\"Comment 8\"")
+		(comment 9 "NA")
 	)
 	(text_box "${RELEASE_BODY_1.1.0}"
@@
 				(color 0 0 194 1)
 			)
+			(justify right)
 		)
 	)
