File: Revision History.kicad_sch (KiCad schematic)
At the start: 0 parts

Commit message: Updated switcher IC
Changed lines of the file:
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@@
 		(exclude_from_sim no)
 		(at 20.32 35.56 0)
-		(size 63.5 34.29)
+		(size 63.5 40.64)
 		(margins 1.4287 1.4287 1.4287 1.4287)
 		(stroke
@@
 	(text_box "${RELEASE_TITLE_1.0.2}"
 		(exclude_from_sim no)
-		(at 152.4 31.75 0)
+		(at 20.32 114.3 0)
 		(size 63.5 3.81)
 		(margins 1.4287 1.4287 1.4287 1.4287)
@@
 	(text_box "${RELEASE_BODY_1.0.2}"
 		(exclude_from_sim no)
-		(at 152.4 35.56 0)
-		(size 63.5 111.76)
+		(at 20.32 118.11 0)
+		(size 63.5 72.39)
 		(margins 1.4287 1.4287 1.4287 1.4287)
 		(stroke
@@
 		(exclude_from_sim no)
 		(at 20.32 80.01 0)
-		(size 63.5 105.41)
+		(size 63.5 34.29)
 		(margins 1.4287 1.4287 1.4287 1.4287)
 		(stroke
