File: StepUp_module_12to450V.kicad_pcb (KiCad board)
At the start: 2 copper layers, 81.8 x 47.2 mm, 37 parts, among them J1 Screw_Terminal_01x04, Q1 HY1707, Q2 HY1707, Q3 S8050, U1 UC2843A

Commit message: Updated switcher IC
Parts:
- R9: value R -> 13.7m
- TR1: value ~ -> ?
- U1: value UC2843A -> UC3845
- moved U1 0.34 mm to (129.5, 88.5)
Connections:
- TR1 pad 3: GND -> (no net)
